File: DMX-Controller.kicad_sch (KiCad schematic)
At the start: 22 parts, among them J1 DMX_IN, J2 DMX_OUT, J3 DC-005 2.0, SW1 POWER_EN, U1 MAX3430ESA, U3 ESP32_NODEMCU, U4 XL1509-5.0E1

Commit message: chore: fix 3d model
Parts:
- U1: MP MAX485 -> MAX3430ESA
Changed lines of the file:
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@@
 			)
 		)
-		(property "MP" "MAX485"
+		(property "MP" "MAX3430ESA"
 			(at 138.938 27.178 0)
 			(effects
